Commit message: 🎈 perf: 将odom更名为gimbal_odom
与导航系统tf树合并为同一棵树

File: src/rm_gimbal_description/urdf/rm_gimbal.urdf.xacro (robot description, xacro)
@@ -1,11 +1,17 @@
 <?xml version="1.0" encoding="utf-8"?>
-<robot name="rm_gimbal"
+<robot name="sentry_gimbal"
   xmlns:xacro="http://ros.org/wiki/xacro">
   <xacro:arg name="xyz" default="0.10 0 0.05" />
   <xacro:arg name="rpy" default="0 0 0" />
-  <link name="odom" />
+  <link name="base_link" />
+  <link name="gimbal_odom" />
+  <joint name="base_joint" type="fixed">
+    <origin xyz="0 0 0.5" rpy="0 0 0" />
+    <parent link="base_link" />
+    <child link="gimbal_odom" />
+  </joint>
   <link name="gimbal_link" />
   <joint name="gimbal_joint" type="floating">
-    <parent link="odom" />
+    <parent link="gimbal_odom" />
     <child link="gimbal_link" />
   </joint>

Commit message: perf(hik_camera): 添加若干个相机内参

File: src/rm_gimbal_description/urdf/rm_gimbal.urdf.xacro (robot description, xacro)
@@ -24,2 +24,50 @@
   </joint>
 </robot>
+<!-- <robot name="rm_gimbal"
+  xmlns:xacro="http://ros.org/wiki/xacro">
+  <xacro:arg name="xyz" default="0.10 0 0.05" />
+  <xacro:arg name="rpy" default="0 0 0" />
+  <link name="gimbal_yaw" />
+  <link name="gimbal_pitch" />
+  <joint name="gimbal_pitch_joint" type="floating">
+    <parent link="gimbal_yaw" />
+    <child link="gimbal_pitch" />
+  </joint>
+  <link name="front_industrial_camera" />
+  <joint name="camera_joint" type="fixed">
+    <origin xyz="$(arg xyz)" rpy="$(arg rpy)" />
+    <parent link="gimbal_pitch" />
+    <child link="front_industrial_camera" />
+    <axis xyz="0 0 0" />
+  </joint>
+  <link name="camera_optical_frame" />
+  <joint name="camera_optical_joint" type="fixed">
+    <origin xyz="0 0 0" rpy="${-pi/2} 0 ${-pi/2}" />
+    <parent link="front_industrial_camera" />
+    <child link="camera_optical_frame" />
+  </joint>
+</robot> -->
+<!-- <robot name="rm_gimbal"
+  xmlns:xacro="http://ros.org/wiki/xacro">
+  <xacro:arg name="xyz" default="0.10 0 0.05" />
+  <xacro:arg name="rpy" default="0 0 0" />
+  <link name="chassis" />
+  <link name="gimbal_yaw" />
+  <joint name="gimbal_yaw_joint" type="floating">
+    <parent link="chassis" />
+    <child link="gimbal_yaw" />
+  </joint>
+  <link name="gimbal_pitch" />
+  <joint name="gimbal_pitch_joint" type="fixed">
+    <origin xyz="$(arg xyz)" rpy="$(arg rpy)" />
+    <parent link="gimbal_yaw" />
+    <child link="gimbal_pitch" />
+    <axis xyz="0 0 0" />
+  </joint>
+  <link name="front_industrial_camera" />
+  <joint name="camera_optical_joint" type="fixed">
+    <origin xyz="0 0 0" rpy="${-pi/2} 0 ${-pi/2}" />
+    <parent link="gimbal_pitch" />
+    <child link="front_industrial_camera" />
+  </joint>
+</robot> -->

Commit message: 🎈 perf(tracker): try some solve

File: src/rm_gimbal_description/urdf/rm_gimbal.urdf.xacro (robot description, xacro)
@@ -24,50 +24,2 @@
   </joint>
 </robot>
-<!-- <robot name="rm_gimbal"
-  xmlns:xacro="http://ros.org/wiki/xacro">
-  <xacro:arg name="xyz" default="0.10 0 0.05" />
-  <xacro:arg name="rpy" default="0 0 0" />
-  <link name="gimbal_yaw" />
-  <link name="gimbal_pitch" />
-  <joint name="gimbal_pitch_joint" type="floating">
-    <parent link="gimbal_yaw" />
-    <child link="gimbal_pitch" />
-  </joint>
-  <link name="front_industrial_camera" />
-  <joint name="camera_joint" type="fixed">
-    <origin xyz="$(arg xyz)" rpy="$(arg rpy)" />
-    <parent link="gimbal_pitch" />
-    <child link="front_industrial_camera" />
-    <axis xyz="0 0 0" />
-  </joint>
-  <link name="camera_optical_frame" />
-  <joint name="camera_optical_joint" type="fixed">
-    <origin xyz="0 0 0" rpy="${-pi/2} 0 ${-pi/2}" />
-    <parent link="front_industrial_camera" />
-    <child link="camera_optical_frame" />
-  </joint>
-</robot> -->
-<!-- <robot name="rm_gimbal"
-  xmlns:xacro="http://ros.org/wiki/xacro">
-  <xacro:arg name="xyz" default="0.10 0 0.05" />
-  <xacro:arg name="rpy" default="0 0 0" />
-  <link name="chassis" />
-  <link name="gimbal_yaw" />
-  <joint name="gimbal_yaw_joint" type="floating">
-    <parent link="chassis" />
-    <child link="gimbal_yaw" />
-  </joint>
-  <link name="gimbal_pitch" />
-  <joint name="gimbal_pitch_joint" type="fixed">
-    <origin xyz="$(arg xyz)" rpy="$(arg rpy)" />
-    <parent link="gimbal_yaw" />
-    <child link="gimbal_pitch" />
-    <axis xyz="0 0 0" />
-  </joint>
-  <link name="front_industrial_camera" />
-  <joint name="camera_optical_joint" type="fixed">
-    <origin xyz="0 0 0" rpy="${-pi/2} 0 ${-pi/2}" />
-    <parent link="gimbal_pitch" />
-    <child link="front_industrial_camera" />
-  </joint>
-</robot> -->

Commit message: 🐞 fix(tracker): fix a tf bug

File: src/rm_gimbal_description/urdf/rm_gimbal.urdf.xacro (robot description, xacro)
@@ -17,9 +17,9 @@
     <axis xyz="0 0 0" />
   </joint>
-  <link name="camera_optical_frame" />
+  <link name="fonr_industrial_camera" />
   <joint name="camera_optical_joint" type="fixed">
     <origin xyz="0 0 0" rpy="${-pi/2} 0 ${-pi/2}" />
     <parent link="camera_link" />
-    <child link="camera_optical_frame" />
+    <child link="fonr_industrial_camera" />
   </joint>
 </robot>

Commit message: ✨ feat(串口、弹道解算): 添加虚拟串口和弹道解算节点
虚拟串口节点的作用是替代原来的串口，提供自瞄需要的云台姿态。弹道解算节点根据识别到的target来计算出云台的补偿后的目标姿态。

File: src/rm_gimbal_description/urdf/rm_gimbal.urdf.xacro (robot description, xacro)
@@ -17,9 +17,9 @@
     <axis xyz="0 0 0" />
   </joint>
-  <link name="fonr_industrial_camera" />
+  <link name="camera_optical_frame" />
   <joint name="camera_optical_joint" type="fixed">
     <origin xyz="0 0 0" rpy="${-pi/2} 0 ${-pi/2}" />
     <parent link="camera_link" />
-    <child link="fonr_industrial_camera" />
+    <child link="camera_optical_frame" />
   </joint>
 </robot>
